File: electronics/pcb/control_board/control_board.kicad_sch (KiCad schematic)
At the start: 31 parts, among them J1 Motor M1X, J10 Test (Analog Discovery), J2 Motor M1Y, J3 Motor M2X, J4 Motor M2Y, J5 12V IN, J6 12V IN 5.5x2.1, J7 Laser, J8 PD reference, J9 PD output, U1 TMC2209 M1X (addr 0), U2 TMC2209 M1Y (addr 1), U3 TMC2209 M2X (addr 2), U4 TMC2209 M2Y (addr 3)

Commit message: Keep the TMC2209 screw terminals on the control board
The breakouts now plug in by their 10-pin logic header only and keep their
screw terminals. The top pair sits with its terminals on the top edge and
the bottom pair on the bottom edge, so the motor and VM wires come in from
outside the board. Two M2 standoff holes sit under each breakout's
terminal-end mounting holes.

The JST-XH motor plugs are gone. A 2-pin VM plug (J1-J4) and a 100 uF
capacitor next to each driver feed the breakout's VM terminals over a
short lead. The power input, test header and VM plugs moved into the
middle of the board, which is still 100 x 100 mm.

A thin ground tree under the pours keeps every pour piece connected.
The socket footprints now carry the female header 3D models, so the
render shows them. ERC and DRC with schematic parity report no errors.
The wiring docs, system diagram and BOM are updated to match.
Parts:
- J1: value Motor M1X -> VM M1X; footprint Connector_JST:JST_XH_B4B-XH-A_1x04_P2.50mm_Vertical -> Connector_JST:JST_XH_B2B-XH-A_1x02_P2.50mm_Vertical; symbol Connector_Generic:Conn_01x04 -> Connector_Generic:Conn_01x02
- J2: value Motor M1Y -> VM M1Y; footprint Connector_JST:JST_XH_B4B-XH-A_1x04_P2.50mm_Vertical -> Connector_JST:JST_XH_B2B-XH-A_1x02_P2.50mm_Vertical; symbol Connector_Generic:Conn_01x04 -> Connector_Generic:Conn_01x02
- J3: value Motor M2X -> VM M2X; footprint Connector_JST:JST_XH_B4B-XH-A_1x04_P2.50mm_Vertical -> Connector_JST:JST_XH_B2B-XH-A_1x02_P2.50mm_Vertical; symbol Connector_Generic:Conn_01x04 -> Connector_Generic:Conn_01x02
- J4: value Motor M2Y -> VM M2Y; footprint Connector_JST:JST_XH_B4B-XH-A_1x04_P2.50mm_Vertical -> Connector_JST:JST_XH_B2B-XH-A_1x02_P2.50mm_Vertical; symbol Connector_Generic:Conn_01x04 -> Connector_Generic:Conn_01x02
Connections:
- net +12V: now also J1.1 (Pin_1), J2.1 (Pin_1), J3.1 (Pin_1), J4.1 (Pin_1); no longer U1.16 (VM), U2.16 (VM), U3.16 (VM), U4.16 (VM)
- net GND: now also J1.2 (Pin_2), J2.2 (Pin_2), J3.2 (Pin_2), J4.2 (Pin_2); no longer U1.15 (GND), U2.15 (GND), U3.15 (GND), U4.15 (GND)
- removed net M1X_1A: J1.1 (Pin_1), U1.12 (1A)
- removed net M1X_1B: J1.2 (Pin_2), U1.11 (1B)
- removed net M1X_2A: J1.3 (Pin_3), U1.13 (2A)
- removed net M1X_2B: J1.4 (Pin_4), U1.14 (2B)
- removed net M1Y_1A: J2.1 (Pin_1), U2.12 (1A)
- removed net M1Y_1B: J2.2 (Pin_2), U2.11 (1B)
- removed net M1Y_2A: J2.3 (Pin_3), U2.13 (2A)
- removed net M1Y_2B: J2.4 (Pin_4), U2.14 (2B)
- removed net M2X_1A: J3.1 (Pin_1), U3.12 (1A)
- removed net M2X_1B: J3.2 (Pin_2), U3.11 (1B)
- removed net M2X_2A: J3.3 (Pin_3), U3.13 (2A)
- removed net M2X_2B: J3.4 (Pin_4), U3.14 (2B)
- removed net M2Y_1A: J4.1 (Pin_1), U4.12 (1A)
- removed net M2Y_1B: J4.2 (Pin_2), U4.11 (1B)
- removed net M2Y_2A: J4.3 (Pin_3), U4.13 (2A)
- removed net M2Y_2B: J4.4 (Pin_4), U4.14 (2B)
Other:
- note added: "Driver UART addresses from MS1/MS2: U1 0, U2 1, U3 2, U4 3. The breakouts keep their screw terminals: motors wire straight into them, and J1-J4 feed each breakout's VM +/- terminals over a short 2-wire lead."
- note removed: "Driver UART addresses from MS1/MS2: U1 0, U2 1, U3 2, U4 3. Fit a 6-pin male header in each breakout's terminal-block holes so the motor outputs and VM plug into the carrier."
